File: KiCad/Bocal_HIDKey.kicad_pcb (KiCad board)
At the start: 2 copper layers, 15.2 x 33.1 mm, 40 parts, among them J1 USB_C_Receptacle_USB2.0, SW1 RESET_SW, SW2 USER_SW, U1 ATmega32U4-MU, Y1 Crystal_GND24_Small

Commit message: .
Parts:
- D1: footprint _mylib:IP4220CZ6 -> _chips:IP4220CZ6
- D2, D3: footprint _kicad_selfmadeStandartFootprint:LED_SMD_0402 -> LED_SMD:LED_0402_1005Metric_Pad0.77x0.64mm_HandSolder
- moved D2 0.25 mm to (182.1, 83.3)
- moved D3 0.25 mm to (177.2, 83.3)

Commit message: .
Parts:
- removed the R2 at (180.5, 83.3)
- moved R2 1.19 mm to (180.0, 83.3)
- moved D3 0.56 mm to (177.7, 83.3)
- renumbered ISCP6 to GND, ISCP1 to MISO, ISCP4 to MOSI, ISCP5 to RESET, ISCP3 to SCK, ISCP2 to V+
Routing:
- net Net-(J1-PadB5): track 3.02 -> 0.00 mm
