File: KiCad/Bocal_HIDKey.kicad_sch (KiCad schematic)
At the start: 37 parts, among them J1 USB_C_Receptacle_USB2.0, SW1 RESET_SW, SW2 USER_SW, U1 ATmega32U4-MU, Y1 Crystal_GND24_Small

Commit message: .
Parts:
- added R14: 1M, Resistor_SMD:R_0402_1005Metric_Pad0.72x0.64mm_HandSolder, symbol Device:R
- renumbered R9 to R10, R10 to R11, R11 to R12, R12 to R13, R2 to R3, R3 to R4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
Connections:
- net GND: now also R14.1
- net at J1.S1 (SHIELD), R1.2: now also R14.2
Other:
- moved on the sheet: R1
